File: Business_Card/Business_Card.brd (EAGLE design)
At the start: 85 x 55 mm, 5 parts

Commit message: final submit for SAMARTH
Parts:
- moved R1 0.60 mm to (46.0, 42.5)
- moved C1 0.10 mm to (39.5, 42.5)
- moved U$1 0.10 mm to (42.5, 42.5)
Routing:
- net N$7: track 13.5 -> 15.0 mm
- net LED2: track 10.8 -> 11.6 mm
- net ANTENNA_2: track 6.75 -> 7.34 mm
Changed lines of the file:
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@@
 <elements>
 <element name="U$2" library="PCB_BusinessCard" package="25X48MM_NFC_ANTENNA" value="25X48MM_NFC_ANTENNA" x="42.5" y="27.5" smashed="yes" rot="MR0"/>
-<element name="C1" library="rcl" library_urn="urn:adsk.eagle:library:334" package="C0603" package3d_urn="urn:adsk.eagle:package:23616/2" value="220nf" x="39.4" y="42.5" smashed="yes" rot="MR270">
-<attribute name="POPULARITY" value="73" x="39.4" y="42.5" size="1.778" layer="28" rot="MR270" display="off"/>
-<attribute name="SPICEPREFIX" value="C" x="39.4" y="42.5" size="1.778" layer="28" rot="MR270" display="off"/>
+<element name="C1" library="rcl" library_urn="urn:adsk.eagle:library:334" package="C0603" package3d_urn="urn:adsk.eagle:package:23616/2" value="220nf" x="39.5" y="42.5" smashed="yes" rot="MR270">
+<attribute name="POPULARITY" value="73" x="39.5" y="42.5" size="1.778" layer="28" rot="MR270" display="off"/>
+<attribute name="SPICEPREFIX" value="C" x="39.5" y="42.5" size="1.778" layer="28" rot="MR270" display="off"/>
 </element>
-<element name="U$1" library="PCB_BusinessCard" package="XQFN8" value="NT3H" x="42.4" y="42.5" smashed="yes" rot="MR90"/>
+<element name="U$1" library="PCB_BusinessCard" package="XQFN8" value="NT3H" x="42.5" y="42.5" smashed="yes" rot="MR90"/>
 <element name="LED1" library="led" library_urn="urn:adsk.eagle:library:259" package="CHIPLED_0805" package3d_urn="urn:adsk.eagle:package:15821/2" value="" x="33.04" y="45.04" smashed="yes" rot="R180">
 <attribute name="POPULARITY" value="52" x="33.04" y="45.04" size="1.778" layer="27" rot="R180" display="off"/>
 <attribute name="VALUE" x="30.5" y="46.31" size="1.27" layer="27" rot="R270"/>
 </element>
-<element name="R1" library="rcl" library_urn="urn:adsk.eagle:library:334" package="R0603" package3d_urn="urn:adsk.eagle:package:23555/3" value="" x="45.4" y="42.5" smashed="yes" rot="MR270">
-<attribute name="POPULARITY" value="70" x="45.4" y="42.5" size="1.778" layer="28" rot="MR270" display="off"/>
-<attribute name="SPICEPREFIX" value="R" x="45.4" y="42.5" size="1.778" layer="28" rot="MR270" display="off"/>
-<attribute name="VALUE" x="47.305" y="43.135" size="1.27" layer="28" rot="MR270"/>
+<element name="R1" library="rcl" library_urn="urn:adsk.eagle:library:334" package="R0603" package3d_urn="urn:adsk.eagle:package:23555/3" value="" x="46" y="42.5" smashed="yes" rot="MR270">
+<attribute name="POPULARITY" value="70" x="46" y="42.5" size="1.778" layer="28" rot="MR270" display="off"/>
+<attribute name="SPICEPREFIX" value="R" x="46" y="42.5" size="1.778" layer="28" rot="MR270" display="off"/>
+<attribute name="VALUE" x="47.905" y="43.135" size="1.27" layer="28" rot="MR270"/>
 </element>
 </elements>
@@
 <contactref element="C1" pad="1"/>
 <contactref element="R1" pad="2"/>
-<wire x1="42.9" y1="43.1" x2="42.48" y2="43.1" width="0.3" layer="16"/>
-<wire x1="42.48" y1="43.1" x2="42.4" y2="43.1" width="0.3" layer="16"/>
-<wire x1="45.4" y1="41.65" x2="43.95" y2="43.1" width="0.3" layer="16"/>
-<wire x1="43.95" y1="43.1" x2="42.9" y2="43.1" width="0.3" layer="16"/>
-<wire x1="39.4" y1="43.35" x2="39.97" y2="43.92" width="0.3" layer="16"/>
-<wire x1="42.3374" y1="43.45025625" x2="42.3374" y2="43.2426" width="0.3" layer="16"/>
-<wire x1="42.3374" y1="43.2426" x2="42.48" y2="43.1" width="0.3" layer="16"/>
-<wire x1="41.86765625" y1="43.92" x2="42.3374" y2="43.45025625" width="0.3" layer="16"/>
-<wire x1="39.97" y1="43.92" x2="41.86765625" y2="43.92" width="0.3" layer="16"/>
+<wire x1="39.5" y1="43.35" x2="40.05" y2="43.9" width="0.2" layer="16"/>
+<wire x1="41.91695" y1="43.9" x2="42.5" y2="43.31695" width="0.2" layer="16"/>
+<wire x1="42.5" y1="43.31695" x2="42.5" y2="43.1" width="0.2" layer="16"/>
+<wire x1="40.05" y1="43.9" x2="41.91695" y2="43.9" width="0.2" layer="16"/>
+<wire x1="42.5" y1="43.1" x2="43" y2="43.1" width="0.3" layer="16"/>
+<wire x1="43" y1="43.1" x2="44.3" y2="43.1" width="0.3" layer="16"/>
+<wire x1="45.75" y1="41.65" x2="46" y2="41.65" width="0.3" layer="16"/>
+<wire x1="44.3" y1="43.1" x2="45.75" y2="41.65" width="0.3" layer="16"/>
 </signal>
 <signal name="LED2">
@@
 <contactref element="U$1" pad="VSS"/>
 <contactref element="LED1" pad="C"/>
-<wire x1="39.4" y1="41.65" x2="36.510615625" y2="41.65" width="0.3" layer="16"/>
+<wire x1="39.5" y1="41.65" x2="36.510615625" y2="41.65" width="0.3" layer="16"/>
 <wire x1="36.510615625" y1="41.65" x2="34.170615625" y2="43.99" width="0.3" layer="16"/>
 <wire x1="34.170615625" y1="43.99" x2="33.04" y2="43.99" width="0.3" layer="1"/>
 <via x="34.170615625" y="43.99" extent="1-16" drill="0.35"/>
-<wire x1="42.4" y1="41.9" x2="42.4" y2="41.612321875" width="0.3" layer="16"/>
-<wire x1="42.4" y1="41.612321875" x2="42.16026875" y2="41.372590625" width="0.3" layer="16"/>
-<wire x1="42.16026875" y1="41.372590625" x2="39.677409375" y2="41.372590625" width="0.3" layer="16"/>
-<wire x1="39.677409375" y1="41.372590625" x2="39.4" y2="41.65" width="0.3" layer="16"/>
+<wire x1="39.677409375" y1="41.372590625" x2="39.5" y2="41.65" width="0.3" layer="16"/>
+<wire x1="42.5" y1="41.9" x2="42.5" y2="41.5" width="0.2" layer="16"/>
+<wire x1="42.1" y1="41.1" x2="42.5" y2="41.5" width="0.2" layer="16"/>
+<wire x1="39.5" y1="41.65" x2="40.05" y2="41.1" width="0.2" layer="16"/>
+<wire x1="40.05" y1="41.1" x2="42.1" y2="41.1" width="0.2" layer="16"/>
 </signal>
 <signal name="N$7">
 <contactref element="R1" pad="1"/>
 <contactref element="LED1" pad="A"/>
-<wire x1="45.4" y1="43.35" x2="45.35" y2="43.35" width="0.3" layer="16"/>
-<wire x1="45.35" y1="43.35" x2="42.61" y2="46.09" width="0.3" layer="16"/>
-<wire x1="42.61" y1="46.09" x2="34.170615625" y2="46.09" width="0.3" layer="16"/>
+<wire x1="46" y1="43.35" x2="45.75" y2="43.35" width="0.3" layer="16"/>
 <wire x1="34.170615625" y1="46.09" x2="33.04" y2="46.09" width="0.3" layer="1"/>
 <via x="34.170615625" y="46.09" extent="1-16" drill="0.35"/>
+<wire x1="46" y1="43.35" x2="46" y2="44.5" width="0.3" layer="16"/>
+<wire x1="46" y1="44.5" x2="44.41" y2="46.09" width="0.3" layer="16"/>
+<wire x1="44.41" y1="46.09" x2="34.170615625" y2="46.09" width="0.3" layer="16"/>
 </signal>
 <signal name="ANTENNA_1">
 <contactref element="U$2" pad="P$1"/>
 <contactref element="U$1" pad="LA"/>
-<wire x1="42.95" y1="41.9" x2="43.135" y2="41.715" width="0.3" layer="16"/>
-<wire x1="43.135" y1="41.715" x2="43.135" y2="40.835" width="0.3" layer="16"/>
+<wire x1="43.05" y1="41.9" x2="43.135" y2="41.815" width="0.3" layer="16"/>
+<wire x1="43.135" y1="41.815" x2="43.135" y2="40.835" width="0.3" layer="16"/>
 </signal>
 <signal name="ANTENNA_2">
 <contactref element="U$2" pad="P$2"/>
 <contactref element="U$1" pad="LB"/>
-<via x="43.84" y="41.84" extent="1-16" drill="0.35"/>
-<wire x1="43" y1="42.5" x2="43.0726" y2="42.4274" width="0.3" layer="16"/>
-<wire x1="43.0726" y1="42.4274" x2="43.26025625" y2="42.4274" width="0.3" layer="16"/>
-<wire x1="43.26025625" y1="42.4274" x2="43.4374" y2="42.25025625" width="0.3" layer="16"/>
-<wire x1="43.4374" y1="42.25025625" x2="43.4374" y2="42.2426" width="0.3" layer="16"/>
-<wire x1="43.4374" y1="42.2426" x2="43.84" y2="41.84" width="0.3" layer="16"/>
-<wire x1="43.84" y1="39" x2="43.84" y2="41.84" width="0.3" layer="1"/>
-<wire x1="41.865" y1="37.025" x2="43.84" y2="39" width="0.3" layer="1"/>
+<via x="44.24" y="41.54" extent="1-16" drill="0.35"/>
+<wire x1="44.24" y1="39.4" x2="44.24" y2="41.54" width="0.3" layer="1"/>
+<wire x1="41.865" y1="37.025" x2="44.24" y2="39.4" width="0.3" layer="1"/>
+<wire x1="43.1" y1="42.5" x2="43.8" y2="42.5" width="0.2" layer="16"/>
+<wire x1="44.24" y1="42.06" x2="44.24" y2="41.54" width="0.2" layer="16"/>
+<wire x1="43.8" y1="42.5" x2="44.24" y2="42.06" width="0.2" layer="16"/>
 </signal>
 </signals>
